File: Precharge/Precharge.kicad_pcb (KiCad board)
At the start: 2 copper layers, 71.9 x 88.8 mm, 41 parts, among them J1 Conn_02x02_Counter_Clockwise, J2 Conn_02x02_Counter_Clockwise, J3 Molex MicroFit, K1 OMRON-G2RL-2-DC12, Q1 AO3400A, Q2 2N7002, U1 LM393, U2 4N35, U3 NA555D

Commit message: v1.4
Parts:
- added C5: 0.1uF, Capacitor_SMD:C_0603_1608Metric_Pad1.08x0.95mm_HandSolder, F.Cu at (148.4, 89.2)
- added D4: 1N5819, Diode_THT:D_DO-41_SOD81_P7.62mm_Horizontal, F.Cu at (144.5, 71.1)
- added D5: P_C LED, LED_SMD:LED_0805_2012Metric_Pad1.15x1.40mm_HandSolder, F.Cu at (148.3, 107.7)
- added G***: LOGO, LOGO, F.Cu at (106.3, 134.3)
- added J4: Molex MicroFit, Connector_Molex:Molex_Micro-Fit_3.0_43045-0612_2x03_P3.00mm_Vertical, F.Cu at (137.4, 62.4)
- added K2: G5V-2, Relay_THT:Relay_DPDT_Omron_G5V-2, F.Cu at (134.4, 89.7)
- added R22: 1M, Resistor_SMD:R_0603_1608Metric_Pad0.98x0.95mm_HandSolder, F.Cu at (149.6, 74.8)
- added R23: 10K, Resistor_SMD:R_0603_1608Metric_Pad0.98x0.95mm_HandSolder, F.Cu at (145.8, 85.1)
- added R24: 220K, Resistor_SMD:R_0603_1608Metric_Pad0.98x0.95mm_HandSolder, F.Cu at (150.6, 80.4)
- added R25: 33K, Resistor_SMD:R_0603_1608Metric_Pad0.98x0.95mm_HandSolder, F.Cu at (141.7, 85.1)
- added R26: 22K, Resistor_SMD:R_0603_1608Metric_Pad0.98x0.95mm_HandSolder, F.Cu at (143.8, 85.1)
- added R27: 1.8K, Resistor_SMD:R_0603_1608Metric_Pad0.98x0.95mm_HandSolder, F.Cu at (146.1, 107.5)
- added REF**: Symbol_HighVoltage_Triangle_6x6mm_Copper, Symbol:Symbol_HighVoltage_Triangle_6x6mm_Copper, F.Cu at (84.9, 75.9)
- added TP1: TestPoint, Connector_Pin:Pin_D1.0mm_L10.0mm, F.Cu at (76.5, 94.5)
- added TP2: TestPoint, Connector_Pin:Pin_D1.0mm_L10.0mm, F.Cu at (76.5, 101.1)
- added TP3: TestPoint, Connector_Pin:Pin_D1.0mm_L10.0mm, F.Cu at (82.0, 59.4)
- added TP5: TestPoint P_C, Connector_Pin:Pin_D1.0mm_L10.0mm, F.Cu at (142.0, 112.8)
- added U4: NE555D, Package_SO:SOIC-8_3.9x4.9mm_P1.27mm, F.Cu at (150.8, 84.3)
- C1: value 10uF -> 0.1 uF
- C2: footprint Capacitor_SMD:C_0805_2012Metric_Pad1.18x1.45mm_HandSolder -> Capacitor_SMD:C_0603_1608Metric_Pad1.08x0.95mm_HandSolder
- C3: value 0.1 uF -> 0.01uF; footprint Capacitor_SMD:C_0805_2012Metric -> Capacitor_SMD:C_0603_1608Metric_Pad1.08x0.95mm_HandSolder
- C4: value 0.01uF -> 10uF; footprint Capacitor_SMD:C_0805_2012Metric_Pad1.18x1.45mm_HandSolder -> Resistor_SMD:R_0805_2012Metric_Pad1.20x1.40mm_HandSolder
- D1, D2: value D_Schottky -> 1N5819
- D3: value 1N4007 -> P_F LED; footprint Diode_THT:D_DO-41_SOD81_P10.16mm_Horizontal -> LED_SMD:LED_0805_2012Metric_Pad1.15x1.40mm_HandSolder
- H1, H2, H3, H4: footprint MountingHole:MountingHole_2.7mm_M2.5_DIN965_Pad -> MountingHole:MountingHole_3.2mm_M3_DIN965
- J1, J2: value Conn_02x02_Counter_Clockwise -> Conn_01x02; footprint Connector_Molex:Molex_Mini-Fit_Jr_5566-04A_2x02_P4.20mm_Vertical -> Connector_Molex:Molex_Mini-Fit_Jr_5566-02A_2x01_P4.20mm_Vertical
- J3: value Molex MicroFit -> Conn_02x03_Counter_Clockwise
- K1: value OMRON-G2RL-2-DC12 -> KT12-1A-40L-THT; footprint Relay_THT:Relay_DPDT_Omron_G6S-2 -> Meder:RELAY_KT12-1A-40L-THT
- Q1: value AO3400A -> 2N7002
- R1, R6: value 220K -> 270K
- R12, R14: value 12K -> 3.3K; footprint Resistor_SMD:R_0603_1608Metric_Pad0.98x0.95mm_HandSolder -> Resistor_SMD:R_2512_6332Metric_Pad1.40x3.35mm_HandSolder
- R13: value 56K -> 3.3K; footprint Resistor_SMD:R_0603_1608Metric_Pad0.98x0.95mm_HandSolder -> Resistor_SMD:R_2512_6332Metric_Pad1.40x3.35mm_HandSolder
- R15: value 56K -> 6.8K
- R16: value 470K -> 4.7K
- R17: value 12K -> 10
- R18: value 10K -> 100K
- R19: value 1M -> 1.8K
- R2: value 56K -> 12K
- R20: value 1.2K -> 10K; footprint Resistor_SMD:R_1206_3216Metric -> Resistor_SMD:R_0603_1608Metric_Pad0.98x0.95mm_HandSolder
- R21: value 27K -> 100K; footprint Resistor_SMD:R_1206_3216Metric -> Resistor_SMD:R_0603_1608Metric_Pad0.98x0.95mm_HandSolder
- R3: value 15K -> 12K
- R4: value 56K -> 330
- R5: value 2.7K -> 15K
- R7: value 5.6K -> 1.5K
- R8: value 270 -> 120; footprint Precharge:HS50 -> Chassis_Resistor:HSA25
- U1: footprint Package_SO:SOIC-8_3.9x4.9mm_P1.27mm -> Package_SO:SOIC-8-N7_3.9x4.9mm_P1.27mm
- U3: value NA555D -> 4N35; footprint Package_SO:SOIC-8_3.9x4.9mm_P1.27mm -> Package_DIP:DIP-6_W7.62mm
- moved H2 106.0 mm to (151.3, 56.6)
- moved H3 106.0 mm to (75.3, 132.6)
- moved J1 94.7 mm to (88.2, 57.9), turned to 90 degrees
- moved J2 91.7 mm to (84.6, 129.5), turned to 90 degrees
- moved C1 85.7 mm to (81.9, 63.1), turned to 180 degrees
- moved R5 77.8 mm to (93.6, 63.2), turned to 0 degrees
- moved U3 66.2 mm to (119.9, 64.5)
- moved R14 64.9 mm to (106.2, 67.1), turned to 0 degrees
- moved U1 64.9 mm to (80.0, 67.3)
- moved R6 61.2 mm to (75.2, 109.5)
- moved R3 58.7 mm to (75.2, 114.8), turned to -90 degrees
- moved R4 53.9 mm to (75.2, 120.1)
- moved R12 47.0 mm to (106.2, 62.2), turned to 180 degrees
- moved C2 43.1 mm to (151.6, 74.8), turned to -90 degrees
- moved R21 38.1 mm to (137.7, 85.1), turned to 90 degrees
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Connections:
- C1 pad 1: Net-(U3-DIS) -> Net-(U1C-V+)
- C1 pad 2: GLV- -> HV-
- C2 pad 1: Net-(U3-TR) -> Net-(U4-TR)
- C3 pad 1: Net-(U1C-V+) -> Net-(U4-CV)
- C3 pad 2: HV- -> GLV-
- C4 pad 1: Net-(U3-CV) -> Net-(U4-DIS)
- D1 pad 1: GLV+ -> /SDC_IN
- D2 pad 1: Net-(D2-K) -> /SDC_IN
- D2 pad 2: /PreCh_Int -> /~{AIR1_Int}
- J1 pad 1: Net-(J1-Pin_1) -> HV-
- J1 pad 2: unconnected-(J1-Pin_2-Pad2) -> HV+
- J2 pad 1: HV+ -> HV-
- J2 pad 2: unconnected-(J2-Pin_2-Pad2) -> Net-(J2-Pin_2)
- J3 pad 1: GLV+ -> /~{AIR1_Int}
- J3 pad 2: unconnected-(J3-Pin_2-Pad2) -> /AIR1
- J3 pad 4: GLV- -> /AIR2
- Q1 pad 3: GLV+ -> /~{AIR1_Int}
- Q2 pad 1: /PreCh_Int -> Net-(D4-A)
- R10 pad 2: Net-(R10-Pad2) -> HV+
- R11 pad 1: Net-(R10-Pad2) -> Net-(R11-Pad1)
- R12 pad 1: Net-(Q1-G) -> Net-(R10-Pad1)
- R13 pad 1: Net-(Q1-G) -> Net-(R11-Pad2)
- R13 pad 2: GLV- -> Net-(R13-Pad2)
- R14 pad 1: GLV+ -> Net-(R12-Pad2)
- R14 pad 2: /PreCh_Int -> Net-(R14-Pad2)
- R15 pad 1: /PreCh_Int -> /Precharge
- R15 pad 2: GLV- -> Net-(R15-Pad2)
- R16 pad 1: GLV+ -> /Precharge
- R16 pad 2: Net-(U3-DIS) -> GLV-
- R17 pad 1: Net-(U3-Q) -> Net-(Q1-G)
- R17 pad 2: Net-(D2-K) -> Net-(R17-Pad2)
- R18 pad 1: GLV+ -> Net-(Q1-G)
- R18 pad 2: Net-(U3-TR) -> GLV-
- R19 pad 1: GLV- -> Net-(D3-A)
- R19 pad 2: Net-(U3-TR) -> /~{AIR1_Int}
- R20 pad 1: /Precharge -> Net-(D4-A)
- R20 pad 2: HV- -> /~{AIR1_Int}
- R21 pad 1: Net-(D3-A) -> Net-(D4-A)
- R21 pad 2: /Precharge -> GLV-
- R3 pad 1: Net-(U1C-V+) -> Net-(U1A--)
- R3 pad 2: HV+ -> Net-(R3-Pad2)
- R4 pad 1: Net-(U1A--) -> Net-(R3-Pad2)
- R4 pad 2: Net-(R4-Pad2) -> HV-
- R5 pad 1: Net-(R4-Pad2) -> Net-(U1C-V+)
- R5 pad 2: HV- -> HV+
- R6 pad 1: Net-(J1-Pin_1) -> Net-(J2-Pin_2)
- R8 pad 1: Net-(D3-K) -> Net-(K1-PadCOM)
- R8 pad 2: Net-(J1-Pin_1) -> Net-(J2-Pin_2)
- R9 pad 1: HV+ -> Net-(R11-Pad1)
- R9 pad 2: Net-(R10-Pad1) -> Net-(K1-PadCOM)
- U2 pad 1: Net-(R11-Pad2) -> Net-(R13-Pad2)
- U2 pad 2: Net-(U1-Pad1) -> HV-
- U2 pad 4: Net-(R12-Pad2) -> Net-(R15-Pad2)
- U2 pad 5: GLV+ -> /SDC_IN
- U3 pad 1: GLV- -> Net-(R14-Pad2)
- U3 pad 2: Net-(U3-TR) -> Net-(U1-Pad1)
- U3 pad 3: Net-(U3-Q) -> unconnected-(U3-NC-Pad3)
- U3 pad 4: GLV+ -> Net-(R17-Pad2)
- U3 pad 5: Net-(U3-CV) -> /SDC_IN
- U3 pad 6: Net-(U3-DIS) -> unconnected-(U3-Pad6)
Routing:
- net /SDC_IN: track 0.00 -> 131.0 mm
- net GLV+: track 113.9 -> 0.00 mm
- net /AIR1: track 0.00 -> 96.3 mm, vias 0 -> 1
- net /AIR2: track 0.00 -> 93.3 mm
- net /AIR1_Con: track 0.00 -> 79.3 mm, vias 0 -> 1
- net /~{AIR1_Int}: track 0.00 -> 66.1 mm
- net (no net): track 65.3 -> 0.00 mm, vias 2 -> 0
- net /PreCh_Int: track 0.00 -> 57.2 mm
- net Net-(J2-Pin_2): track 0.00 -> 54.7 mm
- net Net-(U1C-V+): track 67.9 -> 16.9 mm, vias 2 -> 0
- net Net-(D3-K): track 0.00 -> 50.1 mm
- net Net-(R17-Pad2): track 0.00 -> 42.2 mm
- net Net-(K1-PadCOM): track 0.00 -> 34.0 mm
- net Net-(U1A--): track 27.4 -> 59.9 mm
- net HV-: track 5.42 -> 34.9 mm, vias 328 -> 159
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Other:
- board size 71.9 x 88.8 mm -> 87.1 x 86.1 mm
- board text added: "-"
- board text added: "."
- board text added: "AIR1"
- board text added: "AIR1Int"
- board text added: "AIR2"
- board text added: "Comp+"
- board text added: "Comp_In"
- board text added: "GLV-"
- board text added: "HV LV"
- board text added: "PreChg"
- board text added: "PreInt"
- board text added: "SDC_IN"
- board text added: "To TSAL"
- board text added: "V_Cap"
- board text added: "v1.4"
- board text removed: "GLV+ SDC_IN"
- board text removed: "GLV- AIR1-"
- board text removed: "HV_IN"
- board text removed: "TS GLV"
- board text removed: "TS Out"

Commit message: v1.4.1
Parts:
- C1: footprint Capacitor_SMD:C_0805_2012Metric_Pad1.18x1.45mm_HandSolder -> Capacitor_SMD:C_1206_3216Metric_Pad1.33x1.80mm_HandSolder
- moved D5 0.54 mm to (147.8, 107.7), turned to 90 degrees
- moved R27 0.40 mm to (145.7, 107.6), turned to -90 degrees
- moved D3 0.13 mm to (151.0, 107.7)
Routing:
- net /~{AIR1_Int}: track 66.1 -> 64.3 mm
- net GLV-: vias 33 -> 26

Commit message: v1.5
Routing:
- net HV-: track 35.2 -> 109.1 mm, vias 159 -> 150
- net GLV-: track 2.08 -> 36.0 mm, vias 26 -> 19
- net HV+: track 50.8 -> 64.6 mm
- net Net-(K1-PadCOM): track 34.0 -> 38.2 mm
- net Net-(U1A-+): track 50.3 -> 52.0 mm
- net Net-(D3-A): track 12.9 -> 13.6 mm
- net Net-(R14-Pad2): vias 0 -> 1
Other:
- outline, holes or cut-outs redrawn
- board text added: "v1.5"
- board text removed: "v1.4"

Commit message: v2.0
Parts:
- removed K2: G5V-2, Relay_THT:Relay_DPDT_Omron_G5V-2
- removed TP5: TestPoint P_C, Connector_Pin:Pin_D1.0mm_L10.0mm
- added D6: 1N4937, Diode_THT:D_DO-41_SOD81_P7.62mm_Horizontal, F.Cu at (149.4, 71.1)
- added D7: M7, Diode_SMD:D_SMA_Handsoldering, F.Cu at (113.0, 76.8)
- added R28: 33K, Resistor_SMD:R_0603_1608Metric_Pad0.98x0.95mm_HandSolder, F.Cu at (134.4, 102.3)
- added R29: 22K, Resistor_SMD:R_0603_1608Metric_Pad0.98x0.95mm_HandSolder, F.Cu at (134.4, 104.2)
- added TP4: TestPoint P_C, Connector_Pin:Pin_D1.0mm_L10.0mm, F.Cu at (152.0, 108.0)
- C1: footprint Capacitor_SMD:C_1206_3216Metric_Pad1.33x1.80mm_HandSolder -> Capacitor_SMD:C_0805_2012Metric_Pad1.18x1.45mm_HandSolder
- C4: value 10uF -> 0.1uF; footprint Resistor_SMD:R_0805_2012Metric_Pad1.20x1.40mm_HandSolder -> Capacitor_SMD:C_0603_1608Metric_Pad1.08x0.95mm_HandSolder
- C5: value 0.1uF -> 10uF; footprint Capacitor_SMD:C_0603_1608Metric_Pad1.08x0.95mm_HandSolder -> Resistor_SMD:R_0805_2012Metric_Pad1.20x1.40mm_HandSolder
- D2: value 1N5819 -> P_C LED; footprint Diode_THT:D_DO-41_SOD81_P7.62mm_Horizontal -> LED_SMD:LED_0805_2012Metric_Pad1.15x1.40mm_HandSolder
- D5: value P_C LED -> 1N4937; footprint LED_SMD:LED_0805_2012Metric_Pad1.15x1.40mm_HandSolder -> Diode_THT:D_DO-41_SOD81_P7.62mm_Horizontal
- J3: value Conn_02x03_Counter_Clockwise -> Molex MicroFit
- J4: value Molex MicroFit -> Conn_02x03_Counter_Clockwise
- Q1: value 2N7002 -> AO3400A
- R16: value 4.7K -> 1.8K
- R17: value 10 -> 4.7K
- R23: value 10K -> 33K
- R24: value 220K -> 22K
- R25: value 33K -> 10K
- R26: value 22K -> 220K
- R27: value 1.8K -> 1M
- U1: footprint Package_SO:SOIC-8-N7_3.9x4.9mm_P1.27mm -> Package_SO:SOIC-8_3.9x4.9mm_P1.27mm
- moved J3 62.1 mm to (140.4, 62.6)
- moved J4 59.6 mm to (147.2, 121.2), turned to 90 degrees
- moved D5 37.5 mm to (139.5, 71.1), turned to -90 degrees
- moved D2 34.1 mm to (138.1, 105.2), turned to 90 degrees
- moved C4 17.8 mm to (143.0, 94.3)
- moved R27 17.8 mm to (152.3, 91.1)
- moved R19 13.8 mm to (140.4, 105.2)
- moved C2 10.4 mm to (150.0, 85.1), turned to 90 degrees
- moved R22 10.4 mm to (148.0, 85.1), turned to -90 degrees
- moved D3 8.75 mm to (142.6, 105.2)
- moved U4 8.35 mm to (145.0, 90.4)
- moved C3 7.46 mm to (147.0, 94.3)
- moved R23 6.05 mm to (139.7, 85.1), turned to -90 degrees
- moved Q1 4.92 mm to (149.1, 99.3)
- moved R18 4.92 mm to (149.0, 103.4)
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Connections:
- net /AIR1 renamed /AIR-
- net Net-(U1A-+) renamed /V_Accu
- net Net-(U1A--) renamed /V_Cap
- C4 pad 1: Net-(U4-DIS) -> /SDC_IN
- C5 pad 1: /SDC_IN -> Net-(U4-DIS)
- D2 pad 1: /SDC_IN -> /AIR+_Con
- D2 pad 2: /~{AIR1_Int} -> Net-(D2-A)
- D5 pad 1: /~{AIR1_Int} -> /SDC_IN
- D5 pad 2: Net-(D5-A) -> /AIR+_Con
- J3 pad 1: /~{AIR1_Int} -> GLV-
- J3 pad 4: /AIR2 -> /AIR+_Con
- J3 pad 5: /PreCh_Int -> /AIR+
- J3 pad 6: /Precharge -> /SDC_IN
- J4 pad 1: /AIR2 -> /AIR+
- J4 pad 2: GLV- -> /AIR+_Int
- J4 pad 5: /AIR1_Con -> /PreCh_Int
- J4 pad 6: /SDC_IN -> /Precharge
- K1 pad COM: Net-(K1-PadCOM) -> Net-(D7-A)
- Q1 pad 1: Net-(Q1-G) -> /PreCh_Complt
- Q1 pad 3: /~{AIR1_Int} -> /AIR+_Con
- R16 pad 1: /Precharge -> Net-(D2-A)
- R16 pad 2: GLV- -> /SDC_IN
- R17 pad 1: Net-(Q1-G) -> /Precharge
- R17 pad 2: Net-(R17-Pad2) -> GLV-
- R18 pad 1: Net-(Q1-G) -> /PreCh_Complt
- R19 pad 2: /~{AIR1_Int} -> /AIR+_Con
- R20 pad 2: /~{AIR1_Int} -> /SDC_IN
- R23 pad 1: /SDC_IN -> Net-(D4-A)
- R23 pad 2: Net-(U4-TR) -> /PreCh_Int
- R24 pad 1: /SDC_IN -> /PreCh_Int
- R24 pad 2: Net-(U4-DIS) -> GLV-
- R25 pad 1: Net-(D4-A) -> /SDC_IN
- R25 pad 2: /PreCh_Int -> Net-(U4-TR)
- R26 pad 1: /PreCh_Int -> /SDC_IN
- R26 pad 2: GLV- -> Net-(U4-DIS)
- R27 pad 1: Net-(D5-A) -> Net-(U4-DIS)
- R27 pad 2: /SDC_IN -> GLV-
- R8 pad 1: Net-(K1-PadCOM) -> Net-(D7-K)
- R9 pad 2: Net-(K1-PadCOM) -> Net-(D7-A)
- U1 pad 5: (no net) -> unconnected-(U1B-+-Pad5)
- U1 pad 6: (no net) -> unconnected-(U1B---Pad6)
- U3 pad 4: Net-(R17-Pad2) -> /PreCh_Complt
Routing:
- net /AIR2: track 93.3 -> 0.00 mm
- net /AIR+_Con: track 0.00 -> 87.9 mm, vias 0 -> 2
- net /AIR+: track 0.00 -> 83.3 mm
- net /AIR1_Con: track 79.3 -> 0.00 mm, vias 1 -> 0
- net /~{AIR1_Int}: track 64.3 -> 0.00 mm
- net /PreCh_Complt: track 0.00 -> 61.3 mm
- net Net-(R17-Pad2): track 42.2 -> 0.00 mm
- net Net-(K1-PadCOM): track 38.2 -> 0.00 mm
- net GLV-: track 36.0 -> 0.26 mm, vias 19 -> 28
- net Net-(D7-A): track 0.00 -> 28.1 mm
- net /AIR-: track 96.5 -> 68.6 mm, vias 1 -> 0
- net /AIR+_Int: track 0.00 -> 26.1 mm
- net Net-(U4-DIS): track 11.4 -> 28.6 mm
- net /SDC_IN: track 131.5 -> 116.0 mm, vias 0 -> 2
- net Net-(D4-A): track 19.7 -> 31.7 mm
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Other:
- board text added: "AIR+"
- board text added: "AIR+Con"
- board text added: "AIR+Int"
- board text added: "AIR-"
- board text added: "NO FEAR!"
- board text added: "v2.0"
- board text removed: "AIR1"
- board text removed: "AIR1Int"
- board text removed: "AIR2"
- board text removed: "v1.5"
