File: Precharge/Precharge.kicad_sch (KiCad schematic)
At the start: 56 parts, among them J1 Conn_02x02_Counter_Clockwise, J2 Conn_02x02_Counter_Clockwise, J3 Molex MicroFit, K1 KT12-1A-40L-THT, K2 G5V-2, Q1 2N7002, Q2 2N7002, U1 LM393, U2 4N35, U3 4N35, U4 NE555D

Commit message: v1.4
Parts:
- removed D1: 1N4007, Diode_THT:D_DO-41_SOD81_P10.16mm_Horizontal, symbol Diode:1N4007
- removed D2, D4: D_Schottky, Diode_THT:D_DO-41_SOD81_P7.62mm_Horizontal, symbol Device:D_Schottky
- removed H1, H2, H3, H4: MountingHole, MountingHole:MountingHole_2.7mm_M2.5_DIN965_Pad, symbol Mechanical:MountingHole_Pad
- removed J1, J2: Conn_02x02_Counter_Clockwise, Connector_Molex:Molex_Mini-Fit_Jr_5566-04A_2x02_P4.20mm_Vertical, symbol Connector_Generic:Conn_02x02_Counter_Clockwise
- added D1, D2, D4: 1N5819, Diode_THT:D_DO-41_SOD81_P7.62mm_Horizontal, symbol Diode:1N5819
- added H1, H2, H3, H4: MountingHole, MountingHole:MountingHole_3.2mm_M3_DIN965, symbol Mechanical:MountingHole
- added J1, J2: Conn_01x02, Connector_Molex:Molex_Mini-Fit_Jr_5566-02A_2x01_P4.20mm_Vertical, symbol Connector_Generic:Conn_01x02
- added J4: Molex MicroFit, Connector_Molex:Molex_Micro-Fit_3.0_43045-0612_2x03_P3.00mm_Vertical, symbol Connector_Generic:Conn_02x03_Counter_Clockwise
- C1: footprint Capacitor_SMD:C_0805_2012Metric -> Capacitor_SMD:C_0805_2012Metric_Pad1.18x1.45mm_HandSolder
- C2, C5: footprint Capacitor_SMD:C_0805_2012Metric_Pad1.18x1.45mm_HandSolder -> Capacitor_SMD:C_0603_1608Metric_Pad1.08x0.95mm_HandSolder
- C3: value 0.1uF -> 0.01uF; footprint Capacitor_SMD:C_0805_2012Metric_Pad1.18x1.45mm_HandSolder -> Capacitor_SMD:C_0603_1608Metric_Pad1.08x0.95mm_HandSolder
- C4: value 15uF -> 10uF; footprint Capacitor_THT:CP_Radial_D8.0mm_P3.80mm -> Resistor_SMD:R_0805_2012Metric_Pad1.20x1.40mm_HandSolder
- D3: value LED -> P_F LED
- D5: value LED -> P_C LED
- J3: value Molex MicroFit -> Conn_02x03_Counter_Clockwise
- K1: footprint KT12-1A-40L-THT:RELAY_KT12-1A-40L-THT -> Meder:RELAY_KT12-1A-40L-THT
- R1, R6: value 220K -> 270K
- R15: value 33K -> 6.8K
- R16: value 22K -> 4.7K
- R2, R3: value 56K -> 12K
- R24: value 330K -> 220K
- R4: value 1.8K -> 330
- R7: value 5.6K -> 1.5K
- R8: value 270 -> 120; footprint Precharge:HS50 -> Chassis_Resistor:HSA25
- TP5: value TestPoint -> TestPoint P_C
Connections:
- net GLV-: now also J4.2 (Pin_2), J4.3 (Pin_3); no longer J3.4 (Pin_4)
- net HV+: now also J1.2 (Pin_2)
- net HV-: now also J1.1 (Pin_1), J2.1 (Pin_1)
- net SDC_IN: now also D1.1 (K), D2.1 (K), J4.6 (Pin_6); no longer J3.2 (Pin_2), R19.2
- net at Q2.1 (G), R20.1, R21.1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: now also D4.2 (A)
- net at D3.1 (K), U4.3 (Q): now also D4.1 (K)
- net at K1.COIL1, Q2.3 (D): now also D1.2 (A)
- net at K1.COM, R9.2: now also R8.1
- net at R6.1, R8.2: now also J2.2 (Pin_2)
- net AIR1- renamed AIR1_Con
- net AIR1_Con: now also J4.5 (Pin_5); no longer J3.1 (Pin_1)
- net ~{PreCh_Complt} renamed ~{AIR1_Int}
- net ~{AIR1_Int}: now also J3.1 (Pin_1), R19.2, D2.2 (A)
- new net AIR1: J3.2 (Pin_2), J4.4 (Pin_4)
- new net AIR2: J3.4 (Pin_4), J4.1 (Pin_1)
- no-connect marks 8 -> 4
Other:
- note added: "2.42s"
- note added: "25W"
- note added: "97.4% V_Cap"
- note added: "AIR1_Con is the "negative" lead of the AIR. 12V when SDC is present. Short to GND to activate AIR."
- note added: "DC LINK CAPACITOR"
- note added: "INPUT"
- note added: "Mini-Fit_Jr_02A"
- note added: "To TSAL"
- note added: "~{V_Cap > 97.5% V_Accu}"
- note removed: "5.45s"
- note removed: "50W"
- note removed: "97.5% V_Cap"
- note removed: "AIR1- is the "negative" lead of the AIR. 12V when SDC is present. Short to GND to activate AIR."
- note removed: "Mini-Fit_Jr_04A"
- note removed: "To DC LINK CAPACITOR"

Commit message: v1.4.1
Other:
- note added: "DC-LINK CAPACITOR"
- note added: "~{V_Cap > 97.4% V_Accu}"
- note removed: "DC LINK CAPACITOR"
- note removed: "~{V_Cap > 97.5% V_Accu}"
Changed lines of the file:
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@@
 	(text "Use 1% resistors"
 		(exclude_from_sim no)
-		(at 74.422 135.128 0)
+		(at 74.168 113.792 0)
 		(effects
 			(font
@@
 		)
 	)
-	(text "DC LINK CAPACITOR"
+	(text "DC-LINK CAPACITOR"
 		(exclude_from_sim no)
-		(at 167.64 174.752 0)
+		(at 167.386 170.434 0)
 		(effects
 			(font
@@
 		)
 	)
-	(text "~{V_Cap > 97.5% V_Accu}"
+	(text "~{V_Cap > 97.4% V_Accu}"
 		(exclude_from_sim no)
 		(at 133.858 125.984 0)

Commit message: v2.0
Parts:
- removed D2: 1N5819, Diode_THT:D_DO-41_SOD81_P7.62mm_Horizontal, symbol Diode:1N5819
- removed K2: G5V-2, Relay_THT:Relay_DPDT_Omron_G5V-2, symbol Relay:G5V-2
- removed Q1: 2N7002, Package_TO_SOT_SMD:SOT-23, symbol Transistor_FET:2N7002
- removed R17: 10, Resistor_SMD:R_0603_1608Metric_Pad0.98x0.95mm_HandSolder, symbol Device:R
- removed TP5: TestPoint P_C, Connector_Pin:Pin_D1.0mm_L10.0mm, symbol Connector:TestPoint
- added D5, D6: 1N4937, Diode_THT:D_DO-41_SOD81_P7.62mm_Horizontal, symbol Diode:1N5819
- added D7: M7, Diode_SMD:D_SMA_Handsoldering, symbol Device:D
- added Q1: AO3400A, Package_TO_SOT_SMD:SOT-23, symbol Transistor_FET:AO3400A
- added R27: 1M, Resistor_SMD:R_0603_1608Metric_Pad0.98x0.95mm_HandSolder, symbol Device:R
- added R28: 33K, Resistor_SMD:R_0603_1608Metric_Pad0.98x0.95mm_HandSolder, symbol Device:R
- added R29: 22K, Resistor_SMD:R_0603_1608Metric_Pad0.98x0.95mm_HandSolder, symbol Device:R
- added TP4: TestPoint P_C, Connector_Pin:Pin_D1.0mm_L10.0mm, symbol Connector:TestPoint
- U1: footprint Package_SO:SOIC-8-N7_3.9x4.9mm_P1.27mm -> Package_SO:SOIC-8_3.9x4.9mm_P1.27mm
- renumbered C5 to C4, C4 to C5, D5 to D2, J4 to J3, J3 to J4, R27 to R16, R16 to R17, R25 to R23, R26 to R24, R23 to R25, R24 to R26
Connections:
- net GLV-: now also J3.1 (Pin_1), Q1.2 (S), R27.2, R29.2; no longer J3.2 (Pin_2)
- net SDC_IN: now also R20.2, D5.1 (K)
- net at D4.2 (A), Q2.1 (G), R20.1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: now also D6.2 (A)
- net at C5.1, R26.2, U4.6 (THR)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: now also R27.1
- net V_Cap: now reaches R3.1, R6.2, TP2.1, U1.2 (-)
- net V_Accu: now reaches R1.1, R2.2, TP1.1, U1.3 (+)
- net PreCh_Complt: now reaches R18.1
- net PreCh_Complt: now also U3.4, Q1.1 (G), R28.1, TP4.1
- net at K1.COM, R9.2: now also D7.2 (A); no longer R8.1
- net AIR1 renamed AIR+_Con
- net AIR+_Con: now also D2.1 (K), R19.2, D5.2 (A), D6.1 (K), Q1.3 (D); no longer J4.2 (Pin_2)
- net AIR1_Con renamed AIR+
- net AIR+: now also J4.1 (Pin_1)
- net AIR2 renamed AIR-
- net AIR-: now also J3.2 (Pin_2); no longer J3.1 (Pin_1)
- removed net ~{AIR1_Int}: D2.1 (K), J4.1 (Pin_1), R19.2, R20.2
- new net: D7.1 (K), R8.1
- new net AIR+_Int: J4.2 (Pin_2), R28.2, R29.1
- no-connect marks 4 -> 2
Other:
- note added: "3s"
- note added: "AIR+_Con is the "negative" lead of AIR+. 12V when SDC is present. Short to GND to activate AIR."
- note removed: "2.42s"
- note removed: "97.4% V_Cap"
- note removed: "AIR1_Con is the "negative" lead of the AIR. 12V when SDC is present. Short to GND to activate AIR."
- note removed: "V_Cap"
- moved on the sheet: H1, H2, H3, H4, R18

Commit message: v2.1
Parts:
- removed R27: 1M, Resistor_SMD:R_0603_1608Metric_Pad0.98x0.95mm_HandSolder, symbol Device:R
- added Q3: 2N7002, Package_TO_SOT_SMD:SOT-23, symbol Transistor_FET:2N7002
- added R29: 1M, Resistor_SMD:R_0603_1608Metric_Pad0.98x0.95mm_HandSolder, symbol Device:R
- R8: value 120 -> 150
- renumbered D7 to D1, D1 to D2, D2 to D3, D6 to D4, D3 to D5, D5 to D6, D4 to D7, R28 to R18, R29 to R19, R18 to R20, R19 to R21, R20 to R22, R21 to R23, R22 to R24, R23 to R25, R24 to R26, R25 to R27, R26 to R28
Connections:
- net GLV-: now also Q3.2 (S); no longer C2.2, C3.2, C4.2, C5.2, R24.1, U4.1 (GND)
- net at C5.1, R28.2, U4.6 (THR)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: now also R29.1
- net Precharge_12V: now reaches R15.2, U2.4
- net Precharge_12V: now also Q3.1 (G)
- new net: C2.2, C3.2, C4.2, C5.2, Q3.3 (D), R24.1, R29.2, U4.1 (GND)

Commit message: v2.1
Connections:
- net Comp_Out: now reaches U1.1, U3.2
Other:
- note added: "Precharge Relay Control"
- moved on the sheet: Q1, R20

Commit message: v2.1
Parts:
- removed Q3: 2N7002, Package_TO_SOT_SMD:SOT-23, symbol Transistor_FET:2N7002
- added Q3: AO3400A, Package_TO_SOT_SMD:SOT-23, symbol Transistor_FET:AO3400A
Connections:
- net GLV-: now also Q3.2 (S)
- net Precharge_12V: now also Q3.1 (G)
- net at C2.2, C3.2, C4.2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: now also Q3.3 (D)
Changed lines of the file:
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@@
 	)
 	(junction
-		(at 234.95 105.41)
-		(diameter 0)
-		(color 0 0 0 0)
-	)
-	(junction
 		(at 312.42 97.79)
 		(diameter 0)
@@
 	)
 	(junction
+		(at 229.87 119.38)
+		(diameter 0)
+		(color 0 0 0 0)
+	)
+	(junction
 		(at 350.52 139.7)
 		(diameter 0)
@@
 	)
 	(junction
-		(at 234.95 119.38)
+		(at 215.9 193.04)
 		(diameter 0)
 		(color 0 0 0 0)
 	)
 	(junction
-		(at 215.9 193.04)
+		(at 85.09 48.26)
 		(diameter 0)
 		(color 0 0 0 0)
 	)
 	(junction
-		(at 85.09 48.26)
+		(at 229.87 105.41)
 		(diameter 0)
 		(color 0 0 0 0)
@@
 	)
 	(junction
-		(at 234.95 143.51)
-		(diameter 0)
-		(color 0 0 0 0)
-	)
-	(junction
 		(at 234.95 180.34)
 		(diameter 0)
@@
 	(wire
 		(pts
+			(xy 229.87 158.75) (xy 234.95 158.75)
+		)
+		(stroke
+			(width 0)
+			(type default)
+		)
+	)
+	(wire
+		(pts
 			(xy 210.82 193.04) (xy 215.9 193.04)
 		)
@@
 	(wire
 		(pts
-			(xy 234.95 105.41) (xy 240.03 105.41)
-		)
-		(stroke
-			(width 0)
-			(type default)
-		)
-	)
-	(wire
-		(pts
 			(xy 326.39 152.4) (xy 326.39 151.13)
 		)
@@
 	(wire
 		(pts
-			(xy 234.95 143.51) (xy 234.95 158.75)
-		)
-		(stroke
-			(width 0)
-			(type default)
-		)
-	)
-	(wire
-		(pts
 			(xy 260.35 86.36) (xy 260.35 88.9)
 		)
@@
 	(wire
 		(pts
-			(xy 234.95 143.51) (xy 238.76 143.51)
-		)
-		(stroke
-			(width 0)
-			(type default)
-		)
-	)
-	(wire
-		(pts
 			(xy 350.52 113.03) (xy 350.52 118.11)
 		)
@@
 	(wire
 		(pts
-			(xy 234.95 119.38) (xy 234.95 143.51)
+			(xy 229.87 119.38) (xy 229.87 158.75)
 		)
 		(stroke
@@
 	(wire
 		(pts
-			(xy 234.95 105.41) (xy 234.95 119.38)
+			(xy 229.87 105.41) (xy 229.87 119.38)
 		)
 		(stroke
@@
 	(wire
 		(pts
-			(xy 234.95 97.79) (xy 234.95 105.41)
+			(xy 229.87 97.79) (xy 229.87 105.41)
 		)
 		(stroke
@@
 	(wire
 		(pts
-			(xy 236.22 97.79) (xy 234.95 97.79)
+			(xy 236.22 97.79) (xy 229.87 97.79)
 		)
 		(stroke
@@
 	(wire
 		(pts
+			(xy 234.95 143.51) (xy 234.95 158.75)
+		)
+		(stroke
+			(width 0)
+			(type default)
+		)
+	)
+	(wire
+		(pts
 			(xy 156.21 88.9) (xy 156.21 139.7)
 		)
@@
 	(wire
 		(pts
+			(xy 229.87 105.41) (xy 240.03 105.41)
+		)
+		(stroke
+			(width 0)
+			(type default)
+		)
+	)
+	(wire
+		(pts
 			(xy 256.54 105.41) (xy 312.42 105.41)
 		)
@@
 	(wire
 		(pts
-			(xy 218.44 119.38) (xy 234.95 119.38)
+			(xy 218.44 119.38) (xy 229.87 119.38)
 		)
 		(stroke
@@
 	)
 	(label "AIR+_Con"
-		(at 238.76 143.51 0)
+		(at 234.95 143.51 0)
 		(fields_autoplaced yes)
 		(effects
@@
 	)
 	(symbol
-		(lib_name "2N7002_1")
-		(lib_id "Transistor_FET:2N7002")
-		(at 323.85 146.05 0)
-		(unit 1)
-		(exclude_from_sim no)
-		(in_bom yes)
-		(on_board yes)
-		(dnp no)
-		(fields_autoplaced yes)
-		(property "Reference" "Q3"
-			(at 330.2 144.7799 0)
-			(effects
-				(font
-					(size 1.27 1.27)
-				)
-				(justify left)
-			)
-		)
-		(property "Value" "2N7002"
-			(at 330.2 147.3199 0)
-			(effects
-				(font
-					(size 1.27 1.27)
-				)
-				(justify left)
-			)
-		)
-		(property "Footprint" "Package_TO_SOT_SMD:SOT-23"
-			(at 328.93 147.955 0)
-			(effects
-				(font
-					(size 1.27 1.27)
-					(italic yes)
-				)
-				(justify left)
-				(hide yes)
-			)
-		)
-		(property "Datasheet" "https://www.onsemi.com/pub/Collateral/NDS7002A-D.PDF"
-			(at 328.93 149.86 0)
-			(effects
-				(font
-					(size 1.27 1.27)
-				)
-				(justify left)
-				(hide yes)
-			)
-		)
-		(property "Description" "0.115A Id, 60V Vds, N-Channel MOSFET, SOT-23"
-			(at 323.85 146.05 0)
-			(effects
-				(font
-					(size 1.27 1.27)
-				)
-				(hide yes)
-			)
-		)
-		(pin "2"
-		)
-		(pin "1"
-		)
-		(pin "3"
-		)
-		(instances
-			(project ""
-				(path "/5679ed2e-bac1-400d-bcc5-1297256104b1"
-					(reference "Q3")
-					(unit 1)
-				)
-			)
-		)
-	)
-	(symbol
 		(lib_id "Device:R")
 		(at 212.09 101.6 0)
@@
 					(unit 1)
 				)
+			)
+		)
+	)
+	(symbol
+		(lib_id "Transistor_FET:AO3400A")
+		(at 323.85 146.05 0)
+		(unit 1)
+		(exclude_from_sim no)
+		(in_bom yes)
+		(on_board yes)
+		(dnp no)
+		(fields_autoplaced yes)
+		(property "Reference" "Q3"
+			(at 330.2 144.7799 0)
+			(effects
+				(font
+					(size 1.27 1.27)
+				)
+				(justify left)
+			)
+		)
+		(property "Value" "AO3400A"
+			(at 330.2 147.3199 0)
+			(effects
+				(font
+					(size 1.27 1.27)
+				)
+				(justify left)
+			)
+		)
+		(property "Footprint" "Package_TO_SOT_SMD:SOT-23"
+			(at 328.93 147.955 0)
+			(effects
+				(font
+					(size 1.27 1.27)
+					(italic yes)
+				)
+				(justify left)
+				(hide yes)
+			)
+		)
+		(property "Datasheet" "http://www.aosmd.com/pdfs/datasheet/AO3400A.pdf"
+			(at 328.93 149.86 0)
+			(effects
+				(font
+					(size 1.27 1.27)
+				)
+				(justify left)
+				(hide yes)
+			)
+		)
+		(property "Description" "30V Vds, 5.7A Id, N-Channel MOSFET, SOT-23"
+			(at 323.85 146.05 0)
+			(effects
+				(font
+					(size 1.27 1.27)
+				)
+				(hide yes)
+			)
+		)
+		(pin "1"
+		)
+		(pin "2"
+		)
+		(pin "3"
+		)
+		(instances
+			(project "Precharge"
+				(path "/5679ed2e-bac1-400d-bcc5-1297256104b1"
+					(reference "Q3")
+					(unit 1)
+				)

Commit message: v3.0 coming up
Parts:
- removed C3: 0.01uF, Capacitor_SMD:C_0603_1608Metric_Pad1.08x0.95mm_HandSolder, symbol Device:C
- removed C4: 0.1uF, Capacitor_SMD:C_0603_1608Metric_Pad1.08x0.95mm_HandSolder, symbol Device:C
- removed C5: 10uF, Resistor_SMD:R_0805_2012Metric_Pad1.20x1.40mm_HandSolder, symbol Device:C
- removed D1: M7, Diode_SMD:D_SMA_Handsoldering, symbol Device:D
- removed D7: 1N5819, Diode_THT:D_DO-41_SOD81_P7.62mm_Horizontal, symbol Diode:1N5819
- removed Q2: 2N7002, Package_TO_SOT_SMD:SOT-23, symbol Transistor_FET:2N7002
- removed R24, R29: 1M, Resistor_SMD:R_0603_1608Metric_Pad0.98x0.95mm_HandSolder, symbol Device:R
- removed R27: 10K, Resistor_SMD:R_0603_1608Metric_Pad0.98x0.95mm_HandSolder, symbol Device:R
- removed R28: 220K, Resistor_SMD:R_0603_1608Metric_Pad0.98x0.95mm_HandSolder, symbol Device:R
- removed U4: NE555D, Package_SO:SOIC-8_3.9x4.9mm_P1.27mm, symbol Timer:NE555D
- added 2.7M1: R, Resistor_SMD:R_0603_1608Metric_Pad0.98x0.95mm_HandSolder, symbol Device:R
- added D1: 1n4937, Diode_THT:D_DO-41_SOD81_P7.62mm_Horizontal, symbol Diode:1N5819
- added Q2: AO3400A, Package_TO_SOT_SMD:SOT-23, symbol Transistor_FET:AO3400A
- C2: value 0.1uF -> 6.8uF; footprint Capacitor_SMD:C_0603_1608Metric_Pad1.08x0.95mm_HandSolder -> Capacitor_SMD:C_0805_2012Metric_Pad1.18x1.45mm_HandSolder
- D2: value 1N5819 -> 1n4937
Connections:
- net GLV-: now also C2.2, Q2.2 (S)
- net Precharge_12V: now also 2.7M1.1; no longer Q3.1 (G)
- net at D4.2 (A), R22.1, R23.1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: now also D5.1 (K), Q3.3 (D), Q2.1 (G)
- net at C2.1: now also Q3.1 (G), 2.7M1.2
- net at D2.2 (A), K1.COIL1: now also Q2.3 (D)
- net at K1.COM, R9.2: now also D1.2 (A)
- net at R8.1: now also D1.1 (K)
Other:
- moved on the sheet: Q3
