File: TSAL/TSAL.kicad_pcb (KiCad board)
At the start: 2 copper layers, 87.6 x 58.1 mm, 53 parts, among them J1 Conn_02x03_Counter_Clockwise, J2 Conn_01x02, J3 Conn_02x01, J4 Conn_02x01, Q1 BSS138, Q2 BSS138, Q3 AO3401A, U1 LM358, U10 74HC74, U2 74HC27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

Commit message: Add latest circuit PDFs
Parts:
- added C10: 0.1uF, Capacitor_SMD:C_0603_1608Metric_Pad1.08x0.95mm_HandSolder, F.Cu at (117.7, 42.9)
- added C11: 0.1uF, Capacitor_SMD:C_0603_1608Metric_Pad1.08x0.95mm_HandSolder, F.Cu at (113.8, 42.9)
- added C12: 0.1uF, Capacitor_SMD:C_0603_1608Metric_Pad1.08x0.95mm_HandSolder, F.Cu at (110.0, 42.9)
- added C7: 0.1uF, Capacitor_SMD:C_0603_1608Metric_Pad1.08x0.95mm_HandSolder, F.Cu at (118.1, 33.9)
- added C8: 0.1uF, Capacitor_SMD:C_0603_1608Metric_Pad1.08x0.95mm_HandSolder, F.Cu at (114.2, 33.9)
- added C9: 0.1uF, Capacitor_SMD:C_0603_1608Metric_Pad1.08x0.95mm_HandSolder, F.Cu at (110.3, 33.9)
Routing:
- net /AIR-: track 72.3 -> 92.9 mm, vias 0 -> 1
- net /AIR-_Int: track 59.9 -> 74.8 mm, vias 2 -> 3
- net /PreCh_Int: track 96.2 -> 109.7 mm, vias 3 -> 4
- net /AIR+_Int: track 77.3 -> 90.7 mm, vias 0 -> 1
- net /AIR+: track 72.4 -> 85.5 mm, vias 0 -> 1
- net /Precharge: track 100.6 -> 105.3 mm
- net GLV+: track 134.0 -> 131.6 mm
- net Net-(U2-Pad2): track 4.50 -> 3.24 mm
- net /SCS_Compliance: track 43.0 -> 42.2 mm
- net /5V: track 179.5 -> 178.8 mm
- net Net-(U5-Pad3): track 6.72 -> 6.17 mm
- net GLV-: vias 70 -> 76
