File: FullSystemCircuit/FullSystemCircuit.kicad_sch (KiCad schematic)
At the start: 34 parts, among them J1 HVD, K1 Gigavac GV200, K2 Gigavac GV200, SW1 GLVMS, SW10 Left, SW11 Right, SW2 TS_Activate, SW3 BSPD, SW4 IMD, SW5 TSMS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

Commit message: Pushing FluuSystemCircuit
Parts:
- added D15: 1N4001, Diode_THT:D_DO-41_SOD81_P10.16mm_Horizontal, symbol Diode:1N4001
- added RV3: APPS2, symbol Device:R_Potentiometer_Trim
- added U1: Brake Pressure Sense, symbol Sensor_Pressure:40PC015G
- added U18: HTFS400-P, Sensor_Current:LEM_HTFS, symbol Sensor_Current:HTFS400-P
Connections:
- net GLV+: now also RV2.1, RV3.1, U1.1 (Vcc)
- net GLV-: now also RV2.3, D15.1 (K), U1.2 (GND)
- net Precharge Circuit/HV+: now reaches F1.2, K1.2
- net Precharge Circuit/HV-: now reaches BT1.2 (-), K2.1
- new net: D15.2 (A), RV3.3
- new net BSPD/SENS2: U1.3 (Vout)
Other:
- added sheet LV PDIST (../PDIST/PDIST.kicad_sch)
- sheet BSPD ports: added SDC_IN, SDC_OUT, SENS1, SENS2; removed none
- sheet Precharge Circuit ports: added HV+, HV-, TS+, TS-; removed none
- sheet TSAL_RED ports: added TS+, TS-; removed none
- note added: "10K Slide Potentiometers"
- note removed: "MOSFET completes this path"
- moved on the sheet: BT1, BT2, BT3, BT4, BT5, BT6, BT7, D11, D12, D13, D14, E1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
