File: TSAL-RED/TSAL-RED.kicad_sch (KiCad schematic)
At the start: 41 parts, among them J10 Conn_01x02, J11 Conn_01x02, J12 Conn_02x03_Counter_Clockwise, J13 Conn_02x01, K4 G5V-2, Q7 2N7002, Q8 AO3401A, U14 LM358, U15 4N35, U16 NE555D

Commit message: Pushing FluuSystemCircuit
Changed lines of the file:
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@@
-		)
-	)
-	(label "TS+"
-		(at 107.95 86.36 0)
-		(effects
-			(font
-				(size 1.27 1.27)
-				(bold yes)
-			)
-			(justify left bottom)
 		)
 	)
@@
 		)
 	)
-	(label "TS-"
-		(at 107.95 99.06 0)
-		(effects
-			(font
-				(size 1.27 1.27)
-				(bold yes)
-			)
-			(justify left bottom)
-		)
-	)
 	(label "5V+_Iso"
 		(at 170.18 209.55 180)
@@
 			)
 			(justify right bottom)
+		)
+	)
+	(hierarchical_label "TS+"
+		(shape input)
+		(at 107.95 82.55 180)
+		(effects
+			(font
+				(size 1.27 1.27)
+			)
+			(justify right)
 		)
 	)
@@
 		)
 	)
+	(hierarchical_label "TS-"
+		(shape input)
+		(at 107.95 101.6 180)
+		(effects
+			(font
+				(size 1.27 1.27)
+			)
+			(justify right)
+		)
+	)
