File: TSAL-RED/TSAL-RED.kicad_pcb (KiCad board)
At the start: 2 copper layers, 81.9 x 61.6 mm, 42 parts, among them J1 Conn_01x02, J2 Conn_01x02, J5 Conn_02x01, J6 Conn_02x03_Counter_Clockwise, K1 G5V-2, Q1 2N7002, Q2 AO3401A, U1 LM358, U2 4N35, U3 NE555D

Commit message: Precharge modifications
Parts:
- moved R4 15.3 mm to (55.0, 111.5), turned to 90 degrees
Connections:
- D2 pad 1: GLV+ -> AIR+_Sup
- D2 pad 2: HVD_SDC_IN -> TSAC_GLV-
- J6 pad 3: /GRN+ -> GLV-
- J6 pad 4: GLV- -> TSAC_GLV-
- J6 pad 5: HVD_SDC_IN -> AIR+_Sup
- K1 pad 1: HVD_SDC_IN -> TSAC_GLV-
- K1 pad 16: GLV+ -> AIR+_Sup
Routing:
- net AIR+_Sup: track 0.00 -> 36.4 mm
- net TSAC_GLV-: track 0.00 -> 30.9 mm
- net TS+: track 108.2 -> 80.0 mm
- net HVD_SDC_IN: track 26.0 -> 0.00 mm
- net Net-(R4-Pad1): track 41.2 -> 26.0 mm
- net GLV+: track 72.0 -> 66.2 mm
- net /GRN+: track 42.5 -> 39.5 mm
- net GLV-: vias 22 -> 21
Other:
- board text added: "V1.4"
- board text removed: "V1.3"

Commit message: Add PDIST
Parts:
- added R15: 270, Resistor_SMD:R_1206_3216Metric_Pad1.30x1.75mm_HandSolder, F.Cu at (90.7, 94.3)
- R28: value 910 -> 180
Connections:
- R2 pad 2: TS- -> Net-(R15-Pad1)
Routing:
- net TS-: track 9.07 -> 0.00 mm
- net Net-(R15-Pad1): track 0.00 -> 3.18 mm
Other:
- board text added: "V1.5"
- board text removed: "V1.4"
Changed lines of the file:
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@@
 	(net 31 "AIR+_Sup")
 	(net 32 "TSAC_GLV-")
+	(net 33 "Net-(R15-Pad1)")
 	(footprint "Diode_THT:D_DO-41_SOD81_P7.62mm_Horizontal"
 		(layer "F.Cu")
@@
 		)
 	)
+	(footprint "Resistor_SMD:R_1206_3216Metric_Pad1.30x1.75mm_HandSolder"
+		(layer "F.Cu")
+		(at 90.749786 94.314214 -90)
+		(descr "Resistor SMD 1206 (3216 Metric), square (rectangular) end terminal, IPC-7351 nominal with elongated pad for handsoldering. (Body size source: IPC-SM-782 page 72, https://www.pcb-3d.com/wordpress/wp-content/uploads/ipc-sm-782a_amendment_1_and_2.pdf), generated with kicad-footprint-generator")
+		(tags "resistor handsolder")
+		(property "Reference" "R15"
+			(at 0.05 1.85 90)
+			(layer "F.SilkS")
+			(effects
+				(font
+					(size 1 1)
+					(thickness 0.15)
+				)
+			)
+		)
+		(property "Value" "270"
+			(at 0 1.83 90)
+			(layer "F.Fab")
+			(effects
+				(font
+					(size 1 1)
+					(thickness 0.15)
+				)
+			)
+		)
+		(property "Datasheet" ""
+			(at 0 0 90)
+			(layer "F.Fab")
+			(hide yes)
+			(effects
+				(font
+					(size 1.27 1.27)
+					(thickness 0.15)
+				)
+			)
+		)
+		(property "Description" "Resistor"
+			(at 0 0 90)
+			(layer "F.Fab")
+			(hide yes)
+			(effects
+				(font
+					(size 1.27 1.27)
+					(thickness 0.15)
+				)
+			)
+		)
+		(property ki_fp_filters "R_*")
+		(sheetname "/")
+		(sheetfile "TSAL-RED.kicad_sch")
+		(attr smd)
+		(fp_line
+			(start -0.727064 0.91)
+			(end 0.727064 0.91)
+			(stroke
+				(width 0.12)
+				(type solid)
+			)
+			(layer "F.SilkS")
+		)
+		(fp_line
+			(start -0.727064 -0.91)
+			(end 0.727064 -0.91)
+			(stroke
+				(width 0.12)
+				(type solid)
+			)
+			(layer "F.SilkS")
+		)
+		(fp_line
+			(start -2.45 1.13)
+			(end -2.45 -1.13)
+			(stroke
+				(width 0.05)
+				(type solid)
+			)
+			(layer "F.CrtYd")
+		)
+		(fp_line
+			(start 2.45 1.13)
+			(end -2.45 1.13)
+			(stroke
+				(width 0.05)
+				(type solid)
+			)
+			(layer "F.CrtYd")
+		)
+		(fp_line
+			(start -2.45 -1.13)
+			(end 2.45 -1.13)
+			(stroke
+				(width 0.05)
+				(type solid)
+			)
+			(layer "F.CrtYd")
+		)
+		(fp_line
+			(start 2.45 -1.13)
+			(end 2.45 1.13)
+			(stroke
+				(width 0.05)
+				(type solid)
+			)
+			(layer "F.CrtYd")
+		)
+		(fp_line
+			(start -1.6 0.8)
+			(end -1.6 -0.8)
+			(stroke
+				(width 0.1)
+				(type solid)
+			)
+			(layer "F.Fab")
+		)
+		(fp_line
+			(start 1.6 0.8)
+			(end -1.6 0.8)
+			(stroke
+				(width 0.1)
+				(type solid)
+			)
+			(layer "F.Fab")
+		)
+		(fp_line
+			(start -1.6 -0.8)
+			(end 1.6 -0.8)
+			(stroke
+				(width 0.1)
+				(type solid)
+			)
+			(layer "F.Fab")
+		)
+		(fp_line
+			(start 1.6 -0.8)
+			(end 1.6 0.8)
+			(stroke
+				(width 0.1)
+				(type solid)
+			)
+			(layer "F.Fab")
+		)
+		(fp_text user "${REFERENCE}"
+			(at 0 0 90)
+			(layer "F.Fab")
+			(effects
+				(font
+					(size 0.8 0.8)
+					(thickness 0.12)
+				)
+			)
+		)
+		(pad "1" smd roundrect
+			(at -1.55 0 270)
+			(size 1.3 1.75)
+			(layers "F.Cu" "F.Mask" "F.Paste")
+			(roundrect_rratio 0.192308)
+			(net 33 "Net-(R15-Pad1)")
+			(pintype "passive")
+		)
+		(pad "2" smd roundrect
+			(at 1.55 0 270)
+			(size 1.3 1.75)
+			(layers "F.Cu" "F.Mask" "F.Paste")
+			(roundrect_rratio 0.192308)
+			(net 5 "TS-")
+			(pintype "passive")
+			(clearance 0.2)
+			(thermal_bridge_width 1)
+		)
+		(embedded_fonts no)
+		(model "${KICAD9_3DMODEL_DIR}/Resistor_SMD.3dshapes/R_1206_3216Metric.wrl"
+			(offset
+				(xyz 0 0 0)
+			)
+			(scale
+				(xyz 1 1 1)
+			)
+			(rotate
+				(xyz 0 0 0)
+			)
+		)
+	)
 	(footprint "Resistor_SMD:R_0603_1608Metric_Pad0.98x0.95mm_HandSolder"
 		(layer "F.Cu")
@@
 			)
 		)
-		(property "Value" "910"
+		(property "Value" "180"
 			(at 0 1.43 0)
 			(layer "F.Fab")
@@
 		(tags "Resistor Axial_DIN0414 series Axial Horizontal pin pitch 15.24mm 2W length 11.9mm diameter 4.5mm")
 		(property "Reference" "R4"
-			(at 7.62 -3.37 90)
+			(at 7.575 -3 90)
 			(layer "F.SilkS")
 			(effects
@@
 			)
 		)
+		(model "/home/evans/Desktop/FBR/TSAL/CAD/0430450212.stp"
+			(offset
+				(xyz 0 -1.5 5)
+			)
+			(scale
+				(xyz 1 1 1)
+			)
+			(rotate
+				(xyz -0 -0 180)
+			)
+		)
 	)
 	(footprint "Connector_Molex:Molex_Mini-Fit_Jr_5566-02A_2x01_P4.20mm_Vertical"
@@
 			(layers "F.Cu" "F.Mask" "F.Paste")
 			(roundrect_rratio 0.192308)
-			(net 5 "TS-")
+			(net 33 "Net-(R15-Pad1)")
 			(pintype "passive")
 		)
@@
 		)
 	)
-	(gr_text "V1.4"
+	(gr_text "V1.5"
 		(at 112.460786 119.284214 0)
 		(layer "F.SilkS")
@@
 		(net 4)
 	)
-	(segment
-		(start 92.846572 89.45)
-		(end 96.884072 93.4875)
-		(width 0.6096)
-		(layer "F.Cu")
-		(net 5)
-	)
-	(segment
-		(start 92.185786 89.45)
-		(end 92.846572 89.45)
-		(width 0.6096)
-		(layer "F.Cu")
-		(net 5)
-	)
-	(segment
-		(start 96.884072 93.4875)
-		(end 99.4575 93.4875)
-		(width 0.6096)
-		(layer "F.Cu")
-		(net 5)
-	)
-	(segment
-		(start 92.185786 89.45)
-		(end 92.310786 89.45)
-		(width 0.6096)
-		(layer "F.Cu")
-		(net 5)
-	)
 	(via
 		(at 79.230786 93.535214)
@@
 	)
 	(segment
-		(start 86.510786 66.314214)
-		(end 83.235786 63.039214)
-		(width 0.3048)
-		(layer "F.Cu")
-		(net 6)
-	)
-	(segment
-		(start 89.620786 89.464214)
-		(end 88.170786 89.464214)
+		(start 88.599786 104.995214)
+		(end 88.090786 105.504214)
 		(width 0.3048)
 		(layer "F.Cu")
@@
 	)
 	(segment
-		(start 89.620786 103.974214)
-		(end 88.090786 105.504214)
-		(width 0.3048)
+		(start 76.849786 113.089214)
+		(end 84.434786 105.504214)
+		(width 0.6096)
 		(layer "F.Cu")
 		(net 6)
 	)
 	(segment
-		(start 76.849786 113.089214)
-		(end 84.434786 105.504214)
-		(width 0.6096)
+		(start 87.449786 88.743214)
+		(end 87.449786 67.253214)
+		(width 0.3048)
 		(layer "F.Cu")
 		(net 6)
 	)
 	(segment
-		(start 86.510786 87.804214)
-		(end 86.510786 66.314214)
+		(start 88.599786 90.485214)
+		(end 88.599786 104.995214)
 		(width 0.3048)
 		(layer "F.Cu")
@@
 	)
 	(segment
-		(start 89.285786 89.45)
-		(end 89.071572 89.45)
+		(start 89.620786 89.464214)
+		(end 88.170786 89.464214)
 		(width 0.3048)
 		(layer "F.Cu")
@@
 	(segment
 		(start 88.170786 89.464214)
-		(end 86.510786 87.804214)
+		(end 87.449786 88.743214)
+		(width 0.3048)
+		(layer "F.Cu")
+		(net 6)
+	)
+	(segment
+		(start 89.285786 89.45)
+		(end 89.071572 89.45)
 		(width 0.3048)
 		(layer "F.Cu")
@@
 	)
 	(segment
-		(start 83.235786 63.039214)
-		(end 82.460786 63.039214)
+		(start 87.449786 67.253214)
+		(end 83.235786 63.039214)
 		(width 0.3048)
 		(layer "F.Cu")
@@
 	(segment
 		(start 89.620786 89.464214)
-		(end 89.620786 103.974214)
+		(end 88.599786 90.485214)
 		(width 0.3048)
 		(layer "F.Cu")
@@
 	)
 	(segment
+		(start 83.235786 63.039214)
+		(end 82.460786 63.039214)
+		(width 0.3048)
+		(layer "F.Cu")
+		(net 6)
+	)
+	(segment
 		(start 85.365786 111.039214)
 		(end 82.460786 111.039214)
@@
 		(net 32)
 	)
+	(segment
+		(start 90.749786 92.764214)
+		(end 90.749786 90.886)
+		(width 0.254)
+		(layer "F.Cu")
+		(net 33)
+	)
+	(segment
+		(start 90.749786 90.886)
+		(end 91.667618 89.968168)
+		(width 0.254)
+		(layer "F.Cu")
+		(net 33)
+	)
 	(zone

Commit message: Corrected voltage threshold to 50.4V
Parts:
- R15: value 270 -> 150
- R2: value 10K -> 12K
Connections:
- net /Vin renamed /V_Cap
Changed lines of the file:
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@@
 	(net 9 "Net-(Q1-D)")
 	(net 10 "Net-(Q2-G)")
-	(net 11 "/Vin")
+	(net 11 "/V_Cap")
 	(net 12 "Net-(R3-Pad1)")
 	(net 13 "Net-(R3-Pad2)")
@@
 			)
 		)
-		(property "Datasheet" ""
+		(property "Datasheet" "~"
 			(at 0 0 270)
 			(unlocked yes)
@@
 			)
 		)
-		(property "Datasheet" ""
+		(property "Datasheet" "~"
 			(at 0 0 270)
 			(unlocked yes)
@@
 			)
 		)
-		(property "Datasheet" ""
+		(property "Datasheet" "~"
 			(at 0 0 270)
 			(unlocked yes)
@@
 			(layers "F.Cu" "F.Mask" "F.Paste")
 			(roundrect_rratio 0.192308)
-			(net 11 "/Vin")
+			(net 11 "/V_Cap")
 			(pintype "passive")
 		)
@@
 			)
 		)
-		(property "Datasheet" ""
+		(property "Datasheet" "~"
 			(at 0 0 90)
 			(unlocked yes)
@@
 			)
 		)
-		(property "Datasheet" ""
+		(property "Datasheet" "~"
 			(at 0 0 270)
 			(unlocked yes)
@@
 			)
 		)
-		(property "Datasheet" ""
+		(property "Datasheet" "~"
 			(at 0 0 270)
 			(unlocked yes)
@@
 			)
 		)
-		(property "Datasheet" ""
+		(property "Datasheet" "~"
 			(at 0 0 0)
 			(unlocked yes)
@@
 			)
 		)
-		(property "Datasheet" ""
+		(property "Datasheet" "~"
 			(at 0 0 90)
 			(unlocked yes)
@@
 			)
 		)
-		(property "Datasheet" ""
+		(property "Datasheet" "~"
 			(at 0 0 0)
 			(unlocked yes)
@@
 			)
 		)
-		(property "Datasheet" ""
+		(property "Datasheet" "~"
 			(at 0 0 180)
 			(unlocked yes)
@@
 			)
 		)
-		(property "Datasheet" ""
+		(property "Datasheet" "~"
 			(at 0 0 90)
 			(unlocked yes)
@@
 			)
 		)
-		(property "Datasheet" ""
+		(property "Datasheet" "~"
 			(at 0 0 180)
 			(unlocked yes)
@@
 			)
 		)
-		(property "Value" "270"
+		(property "Value" "150"
 			(at 0 1.83 90)
 			(layer "F.Fab")
@@
 			)
 		)
-		(property "Datasheet" ""
+		(property "Datasheet" "~"
 			(at 0 0 90)
 			(layer "F.Fab")
@@
 			)
 		)
-		(property "Datasheet" ""
+		(property "Datasheet" "~"
 			(at 0 0 90)
 			(unlocked yes)
@@
 			)
 		)
-		(property "Datasheet" ""
+		(property "Datasheet" "~"
 			(at 0 0 90)
 			(unlocked yes)
@@
 			)
 		)
-		(property "Datasheet" ""
+		(property "Datasheet" "~"
 			(at 0 0 180)
 			(unlocked yes)
@@
 			)
 		)
-		(property "Datasheet" ""
+		(property "Datasheet" "~"
 			(at 0 0 180)
 			(unlocked yes)
@@
 			)
 		)
-		(property "Datasheet" ""
+		(property "Datasheet" "~"
 			(at 0 0 90)
 			(unlocked yes)
@@
 			)
 		)
-		(property "Datasheet" ""
+		(property "Datasheet" "~"
 			(at 0 0 90)
 			(unlocked yes)
@@
 			)
 		)
-		(property "Datasheet" ""
+		(property "Datasheet" "~"
 			(at 0 0 0)
 			(unlocked yes)
@@
 			)
 		)
-		(property "Datasheet" ""
+		(property "Datasheet" "~"
 			(at 0 0 180)
 			(unlocked yes)
@@
 			)
 		)
-		(property "Datasheet" ""
+		(property "Datasheet" "~"
 			(at 0 0 180)
 			(unlocked yes)
@@
 			)
 		)
-		(property "Datasheet" ""
+		(property "Datasheet" "~"
 			(at 0 0 270)
 			(unlocked yes)
@@
 			)
 		)
-		(property "Datasheet" ""
+		(property "Datasheet" "~"
 			(at 0 0 180)
 			(unlocked yes)
@@
 			)
 		)
-		(property "Datasheet" ""
+		(property "Datasheet" "~"
 			(at 0 0 90)
 			(unlocked yes)
@@
 			)
 		)
-		(property "Datasheet" ""
+		(property "Datasheet" "~"
 			(at 0 0 180)
 			(unlocked yes)
@@
 			)
 		)
-		(property "Datasheet" ""
+		(property "Datasheet" "~"
 			(at 0 0 90)
 			(unlocked yes)
@@
 			)
 		)
-		(property "Datasheet" ""
+		(property "Datasheet" "~"
 			(at 0 0 0)
 			(unlocked yes)
@@
 			)
 		)
-		(property "Datasheet" ""
+		(property "Datasheet" "~"
 			(at 0 0 270)
 			(unlocked yes)
@@
 			)
 		)
-		(property "Datasheet" ""
+		(property "Datasheet" "~"
 			(at 0 0 180)
 			(unlocked yes)
@@
 			)
 		)
-		(property "Datasheet" ""
+		(property "Datasheet" "~"
 			(at 0 0 0)
 			(unlocked yes)
@@
 			(layers "F.Cu" "F.Mask" "F.Paste")
 			(roundrect_rratio 0.25)
-			(net 11 "/Vin")
+			(net 11 "/V_Cap")
 			(pinfunction "-")
 			(pintype "input")
@@
 			)
 		)
-		(property "Value" "10K"
+		(property "Value" "12K"
 			(at 0 1.82 90)
 			(layer "F.Fab")
@@
 			)
 		)
-		(property "Datasheet" ""
+		(property "Datasheet" "~"
 			(at 0 0 270)
 			(unlocked yes)
@@
 			(layers "F.Cu" "F.Mask" "F.Paste")
 			(roundrect_rratio 0.192308)
-			(net 11 "/Vin")
+			(net 11 "/V_Cap")
 			(pintype "passive")
 		)

Commit message: Save corrupted files and new modifications
Parts:
- removed K1: G5V-2, Relay_THT:Relay_DPDT_Omron_G5V-2
- added K2: G2RL-1-E, Relay_THT:Relay_DPDT_Omron_G2RL-2, F.Cu at (112.5, 93.7)
- D2: value 1n4937 -> 1N4148; footprint Diode_THT:D_DO-41_SOD81_P7.62mm_Horizontal -> Diode_THT:D_DO-35_SOD27_P7.62mm_Horizontal
- moved R15 6.80 mm to (91.8, 87.6)
- moved R1 5.51 mm to (89.2, 82.4)
- moved R2 5.51 mm to (91.8, 82.4)
- moved REF** 4.44 mm to (90.5, 71.7)
- moved G*** 3.40 mm to (51.6, 83.7)
- moved H2 3.28 mm to (53.7, 120.4)
- moved J1 3.28 mm to (66.2, 120.0)
- moved R4 3.28 mm to (53.4, 114.4)
- moved R5 3.28 mm to (86.2, 120.2)
- moved R13 2.63 mm to (103.5, 113.4)
- moved J2 2.63 mm to (99.4, 119.9)
- moved R12 2.63 mm to (103.5, 108.1)
- moved H3 2.63 mm to (129.3, 120.2)
- moved R14 1.74 mm to (70.7, 87.3)
- moved H1 1.74 mm to (53.6, 64.3)
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Connections:
- net AIR+_Sup renamed /AIR_Sup+
- net TSAC_GLV- renamed /TSAC_GLV-
Routing:
- net Net-(K2-Pad11): track 34.4 -> 26.7 mm
- net TS-: track 0.00 -> 7.53 mm
- net TS+: track 80.0 -> 83.6 mm
- net Net-(J2-Pin_2): track 7.74 -> 9.56 mm
- net /V_Cap: track 6.35 -> 7.89 mm
- net Net-(R12-Pad1): track 19.4 -> 18.3 mm
- net Net-(R15-Pad1): track 3.18 -> 2.10 mm
- net /AIR_Sup+: track 36.4 -> 35.8 mm
Other:
- board size 81.9 x 61.6 mm -> 83.5 x 64.7 mm
